File: pclptcnc.sch (KiCad schematic (older format))
At the start: 247 parts, among them P1 ARK825A-3, P3 ARK825A-4, P4 ARK825A-3, P5 ARK825A-3, P6 ARK825A-3, P7 ARK825A-3, P8 ARK825A-3, Q1 BC807-40, Q10 BC807-40, Q11 BC807-40, Q12 BC807-40, Q13 BC807-40, Q14 BC807-40, Q15 BC807-40, Q16 BC807-40, Q17 BC807-40, Q18 BC807-40, Q2 BC807-40, Q3 BC807-40, Q4 BC807-40, Q5 BC807-40, Q6 BC807-40, Q7 BC807-40, Q8 BC807-40, Q9 BC807-40, U1 74LVC1G3157GW, U10 SN74LVC2G17, U11 74HCT14, U12 SN74LVC2G17, U13 74HCT14, U2 HCPL2630, U3 HCPL2630, U4 HCPL2630, U5 HCPL2630, U6 HCPL2630, U7 HCPL2630, U8 74HCT14, U9 74HCT14, j1 DB25, j2 DB25

Commit message: revised first PCB version
Parts:
- removed R111, R112, R113, R114, R115, R116, R117, R118, R119, R120, R121, R122, R123, R3, R4, R5, R6, R7: 100K, SM0805, symbol R_SFP
- added R111, R112, R113, R114, R115, R116, R117, R118, R119, R120, R121, R122, R7: 100K, SM0805, symbol R
- R10, R100, R101, R102, R103, R104, R105, R106, R107, R108, R109, R11, R110, R12, R13, R14, R15, R16, R17, R18, R19, R2, R20, R21, R22, R23, R24, R25, R26, R27, R28, R29, R30, R31, R32, R33, R34, R35, R36, R37, R38, R39, R40, R41, R42, R43, R44, R45, R46, R47, R48, R49, R50, R51, R52, R53, R54, R55, R56, R57, R58, R59, R60, R61, R62, R63, R64, R65, R66, R67, R68, R69, R70, R71, R72, R73, R74, R75, R76, R77, R78, R79, R80, R81, R82, R83, R84, R85, R86, R87, R88, R89, R9, R90, R91, R92, R93, R94, R95, R96, R97, R98, R99, R_LED1, R_LED10, R_LED11, R_LED12, R_LED13, R_LED14, R_LED15, R_LED16, R_LED17, R_LED18, R_LED19, R_LED2, R_LED20, R_LED3, R_LED4, R_LED5, R_LED6, R_LED7, R_LED8, R_LED9: symbol R_SFP -> R
- R8: value 180 -> 2K7; symbol R_SFP -> R
Connections:
- net CTRL_SRC: now also R2.2; no longer R2.1
- net FLTRD_SGNL1: now also MUX1.4 (Za); no longer MUX1.9 (Zd)
- net FLTRD_SGNL11: now also MUX3.7 (Zb); no longer MUX3.9 (Zd)
- net FLTRD_SGNL12: now also MUX3.9 (Zd); no longer MUX3.7 (Zb)
- net FLTRD_SGNL2: now also MUX1.12 (Zc); no longer MUX1.7 (Zb)
- net FLTRD_SGNL3: now also MUX1.7 (Zb); no longer MUX1.12 (Zc)
- net FLTRD_SGNL4: now also MUX1.9 (Zd); no longer MUX1.4 (Za)
- net FLTRD_SGNL5: now also MUX2.4 (Za); no longer MUX2.9 (Zd)
- net FLTRD_SGNL6: now also MUX2.12 (Zc); no longer MUX2.7 (Zb)
- net FLTRD_SGNL7: now also MUX2.7 (Zb); no longer MUX2.12 (Zc)
- net FLTRD_SGNL8: now also MUX2.9 (Zd); no longer MUX2.4 (Za)
- net GND: now also C1.2, C2.2, C3.2, C4.2, DC/DC1.2 (GND), P1.3, R_LED2.2, TVS1.1 (A), U1.1 (Y1), R111.2, R112.2, R113.2, R114.2, R115.2, R116.2, R117.2, R118.2, R119.2, R120.2, R121.2, R122.2, R7.2; no longer C5.2, C6.2, C7.2, C8.2, DC/DC1.5 (ISOLATED_GND), R_LED15.1, TVS2.1 (A), U1.3 (Y0)
- net ISOLATED_GND: now also C5.2, C6.2, C7.2, C8.2, DC/DC1.5 (ISOLATED_GND), R_LED15.1, TVS2.1 (A); no longer C1.2, C2.2, C3.2, C4.2, DC/DC1.2 (GND), P1.3, R_LED2.2, TVS1.1 (A)
- net ISOLATED_VCC: now also C5.1, C6.1, C7.1, C8.1, D14.1 (A), F2.2, TVS2.2 (K); no longer C1.1, C2.1, C3.1, C4.1, D1.1 (A), DC/DC1.1 (VCC), F1.2, TVS1.2 (K)
- net ISOLATED_VCC_NFused: now also DC/DC1.7 (ISOLATED_VCC), F2.1; no longer F1.1, P1.1
- net PC1: now also MUX1.6 (I1b); no longer MUX1.13 (I1c)
- net PC10: now also MUX3.13 (I1c); no longer MUX3.10 (I1d)
- net PC11: now also MUX3.6 (I1b); no longer MUX3.13 (I1c)
- net PC12: now also MUX3.10 (I1d), U10.4 (2Y); no longer MUX2.10 (I1d), U11.6 (3Y)
- net PC3: now also MUX1.13 (I1c); no longer MUX1.6 (I1b)
- net PC4: now also U11.2 (1Y); no longer U10.4 (2Y)
- net PC5: now also MUX2.6 (I1b); no longer MUX2.13 (I1c)
- net PC6: now also MUX2.3 (I1a), U11.6 (3Y); no longer MUX2.6 (I1b), U11.2 (1Y)
- net PC7: now also MUX2.13 (I1c); no longer MUX2.3 (I1a)
- net PC8: now also MUX2.10 (I1d), U13.4 (2Y); no longer MUX3.6 (I1b), U13.2 (1Y)
- net PC9: now also U13.2 (1Y); no longer U13.4 (2Y)
- net PC_IN1: now also j2.10; no longer j2.12
- net PC_IN3: now also j2.12; no longer j2.10
- net PC_IN_A1: now also MUX4.9 (Zd); no longer MUX4.7 (Zb)
- net PC_IN_A2: now also U13.8 (4Y); no longer U1.4 (Z)
- net PC_IN_A3: now also MUX4.7 (Zb); no longer MUX4.12 (Zc)
- net PC_IN_A4: now also MUX4.4 (Za); no longer MUX4.9 (Zd)
- net PC_IN_A5: now also MUX4.12 (Zc); no longer MUX4.4 (Za)
- net PC_OUT_A7: now also U11.13 (6A); no longer U11.9 (4A)
- net PC_OUT_A9: now also U11.9 (4A); no longer U11.13 (6A)
- net RC1: now also MUX1.5 (I0b); no longer MUX1.11 (I0d)
- net RC10: now also MUX3.14 (I0c); no longer MUX3.11 (I0d)
- net RC11: now also MUX3.5 (I0b); no longer MUX2.2 (I0a)
- net RC12: now also MUX3.11 (I0d); no longer MUX3.14 (I0c)
- net RC2: now also MUX1.2 (I0a); no longer MUX1.14 (I0c)
- net RC3: now also MUX1.14 (I0c); no longer MUX1.5 (I0b)
- net RC4: now also MUX1.11 (I0d); no longer MUX1.2 (I0a)
- net RC5: now also MUX2.5 (I0b); no longer MUX3.2 (I0a)
- net RC6: now also MUX2.2 (I0a); no longer MUX2.14 (I0c)
- net RC7: now also MUX2.14 (I0c); no longer MUX2.11 (I0d)
- net RC8: now also MUX2.11 (I0d); no longer MUX3.5 (I0b)
- net RC9: now also MUX3.2 (I0a); no longer MUX2.5 (I0b)
- net RCOUT1: now also U8.9 (4A), R7.1; no longer U8.5 (3A)
- net RCOUT10: now also U9.1 (1A), R119.1; no longer U9.5 (3A)
- net RCOUT11: now also R120.1
- net RCOUT12: now also U9.5 (3A), R121.1; no longer U9.1 (1A)
- net RCOUT2: now also U8.11 (5A), R111.1; no longer U8.3 (2A)
- net RCOUT3: now also U8.13 (6A), R112.1; no longer U8.1 (1A)
- net RCOUT4: now also U8.1 (1A), R113.1; no longer U8.9 (4A)
- net RCOUT5: now also U8.3 (2A), R114.1; no longer U8.11 (5A)
- net RCOUT6: now also U8.5 (3A), R115.1; no longer U8.13 (6A)
- net RCOUT7: now also R116.1
- net RCOUT8: now also R117.1
- net RCOUT9: now also R118.1
- net SENSOR_1: now also MUX4.2 (I0a); no longer MUX4.11 (I0d)
- net SENSOR_3: now also MUX4.11 (I0d); no longer MUX4.14 (I0c)
- net SENSOR_4: now also MUX4.14 (I0c), j1.14 (P14); no longer MUX4.2 (I0a), j1.15 (P15)
- net SENSOR_5: now also U1.3 (Y0), j1.15 (P15); no longer U1.1 (Y1), j1.14 (P14)
- net SRC_SEL: now also R122.1
- net VCC: now also C1.1, C2.1, C3.1, C4.1, D1.1 (A), DC/DC1.1 (VCC), F1.2, TVS1.2 (K); no longer C5.1, C6.1, C7.1, C8.1, D14.1 (A), F2.2, TVS2.2 (K)
- net VCC_NFused: now also F1.1, P1.1; no longer DC/DC1.7 (ISOLATED_VCC), F2.1
- net SNSR2: now reaches U13.9 (4A)
- net SNSR2: now also U1.4 (Z)
- net IOSRCTR_BASE: no longer names the net of Q1.1 (B)
- net IOSRCTR_BASE: now also R2.1; no longer R2.2
- net RC_SW_INV renamed PC/RC_SW_inv
- no-connect marks 7 -> 5
Other:
- moved on the sheet: C1, C2, C3, C4, C5, C6, C7, C8, CU1, CU10, CU11, CU12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
